File: SCH_PCB/IGN01A.kicad_pcb (KiCad board)
At the start: 2 copper layers, 0 parts

Commit message: Work on timers PCB started
Parts:
- added C1: 100nF, Capacitors_SMD:C_0805_HandSoldering, F.Cu at (216.4, 134.2)
- added C2: 100nF, Capacitors_SMD:C_0805_HandSoldering, F.Cu at (208.7, 134.2)
- added C3: 22uF/6.3V, Capacitors_SMD:C_0805_HandSoldering, F.Cu at (206.2, 134.2)
- added C4: 100nF, Capacitors_SMD:C_0805_HandSoldering, F.Cu at (120.4, 99.0)
- added C5: 10uF, Capacitors_SMD:C_0805_HandSoldering, F.Cu at (210.2, 156.0)
- added C6: 100nF, Capacitors_SMD:C_0805_HandSoldering, F.Cu at (207.5, 156.0)
- added C7: 100nF, Capacitors_SMD:C_0805_HandSoldering, F.Cu at (204.8, 156.0)
- added D1: 1N4007, Capacitors_SMD:C_0805_HandSoldering, F.Cu at (211.3, 134.2)
- added IC1: ATMEGA328-A, Housings_QFP:TQFP-32_7x7mm_Pitch0.8mm, F.Cu at (191.1, 154.0)
- added J1: PWR, Mlab_Pin_Headers:Angled_1x02, B.Cu at (226.1, 128.4)
- added J2: IGN, Mlab_Pin_Headers:Angled_1x02, B.Cu at (226.1, 122.8)
- added J3: HEADER_1x11, Mlab_Pin_Headers:Angled_1x11, B.Cu at (226.1, 145.4)
- added J5: ISP, Mlab_Pin_Headers:Straight_2x03, F.Cu at (198.3, 136.1)
- added L1: 10uH, Capacitors_SMD:C_0805_HandSoldering, F.Cu at (213.8, 134.2)
- added Q1: IRF7413ZPBF, Housings_SOIC:SOIJ-8_5.3x5.3mm_Pitch1.27mm, F.Cu at (214.2, 124.8)
- added R1: 10k, Capacitors_SMD:C_0805_HandSoldering, F.Cu at (108.3, 113.9)
- added R2: 10k, Capacitors_SMD:C_0805_HandSoldering, F.Cu at (149.0, 107.2)
- added R3: 10k, Capacitors_SMD:C_0805_HandSoldering, F.Cu at (144.6, 102.5)
- added R4, R5: 10k, Capacitors_SMD:C_0805_HandSoldering, F.Cu at (213.8, 172.5)
- added U1: MPL3115A2, SMD_fork:LGA-MPL3115A, F.Cu at (201.2, 156.4)
Routing:
- net VDD: track 0.00 -> 16.3 mm
- net Net-(C7-Pad1): track 0.00 -> 2.69 mm
- net VAA: track 0.00 -> 2.60 mm
- added copper zone on F.Cu, net GND
Other:
- board outline added: 55 x 45 mm
- net class Default: trace_width 0.25 -> 0.5
- net class PWR added: clearance 0.2, trace_width 1.9, via_dia 0.6, via_drill 0.4
- board text added: "+"
- board text added: "-"
- board text added: "A"
- board text added: "C"
- board text added: "GND"
- board text added: "PD3"
- board text added: "PD4"
- board text added: "RST"
- board text added: "RXD"
- board text added: "SCL"
- board text added: "SDA"
- board text added: "TXD"
- board text added: "VDD"

Commit message: pcb added
Parts:
- added R6: 0, Capacitors_SMD:C_1206_HandSoldering, F.Cu at (210.8, 119.7)
- added R7: 0, Capacitors_SMD:C_1206_HandSoldering, F.Cu at (191.8, 109.0)
- added R8: 0, Capacitors_SMD:C_1206_HandSoldering, F.Cu at (186.1, 128.4)
- J3: value HEADER_1x11 -> HEADER_1x09; footprint Mlab_Pin_Headers:Angled_1x11 -> Mlab_Pin_Headers:Angled_1x09
- J5: moved to B.Cu
- moved R1 102.9 mm to (210.8, 123.7), turned to 270 degrees
- moved R4 73.1 mm to (208.7, 99.6), turned to 90 degrees
- moved R3 67.4 mm to (208.5, 123.7), turned to 270 degrees
- moved R2 66.2 mm to (213.1, 123.7), turned to 270 degrees
- moved C4 65.9 mm to (182.0, 122.3)
- moved R5 56.7 mm to (208.5, 116.1), turned to 90 degrees
- moved IC1 41.4 mm to (174.8, 115.9)
- moved D1 39.6 mm to (188.2, 102.1), turned to 0 degrees
- moved C5 37.4 mm to (191.3, 123.7), turned to 180 degrees
- moved C1 35.7 mm to (182.0, 124.7), turned to 0 degrees
- moved C3 34.8 mm to (188.2, 104.4), turned to 0 degrees
- moved C2 34.3 mm to (188.2, 106.7), turned to 0 degrees
- moved C7 32.9 mm to (191.3, 126.0), turned to 180 degrees
- moved L1 32.6 mm to (182.0, 127.0), turned to 0 degrees
- moved J3 32.6 mm to (205.8, 119.9)
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Connections:
- IC1 pad 1: /PD3 -> /OUT
- IC1 pad 2: /PD4 -> /IGN
- IC1 pad 32: /PD2 -> /IN
- J3 pad 3: /PD3 -> /RST
- J3 pad 4: GND -> /RXD
- J3 pad 5: /RXD -> /TXD
- J3 pad 6: /TXD -> /IN
- J3 pad 7: GND -> /OUT
- J3 pad 9: /RST -> GND
- Q1 pad 4: /PD2 -> /IGN
- R4 pad 1: /PD2 -> /IGN
- R5 pad 1: /PD3 -> /IN
Routing:
- net VDD: track 16.3 -> 171.4 mm
- net /RST: track 0.00 -> 86.6 mm
- net GND: track 0.00 -> 64.0 mm
- net /SDA: track 0.00 -> 45.2 mm
- net /SCL: track 0.00 -> 40.7 mm
- net /IGN: track 0.00 -> 40.1 mm
- net /IN: track 0.00 -> 31.2 mm
- net /RXD: track 0.00 -> 29.9 mm
- net /OUT: track 0.00 -> 29.9 mm
- net /TXD: track 0.00 -> 29.2 mm
- net /MOSI: track 0.00 -> 19.6 mm
- net Net-(J2-Pad1): track 0.00 -> 14.0 mm
- net VAA: track 2.60 -> 12.8 mm
- net Net-(J2-Pad2): track 0.00 -> 9.51 mm
- net /MISO: track 0.00 -> 9.21 mm
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Other:
- board size 55 x 45 mm -> 50 x 45 mm
- net class Default: trace_width 0.5 -> 0.25
- net class PWR removed
- rule pad_to_mask_clearance: 0.2 -> 0
- board text added: "IN"
- board text added: "OUT"
- board text removed: "A"
- board text removed: "C"
- board text removed: "GND"
- board text removed: "PD3"
- board text removed: "PD4"
- board text removed: "VDD"
