File: SCH_PCB/IGN01A.sch (KiCad schematic (older format))
At the start: 23 parts, among them IC1 ATMEGA328-A, J1 PWR, J2 IGN, J3 USART, J4 PAD, J5 ISP, Q1 IRF7413ZPBF, U1 MPL3115A2, Y1 Crystal_Small

Commit message: Work on timers PCB started
Parts:
- removed C8, C9: 22pF, Capacitors_SMD:C_0805_HandSoldering, symbol C_Small
- removed J3: USART, Mlab_Pin_Headers:Angled_1x03, symbol HEADER_1x03
- removed J4: PAD, Mlab_Pin_Headers:Angled_1x04, symbol HEADER_1x04
- removed Y1: Crystal_Small, Crystals:Crystal_HC52-U_Vertical, symbol Crystal_Small
- added J?: HEADER_1x11, symbol HEADER_1x11
- added R? (x2): 10k, Capacitors_SMD:C_0805_HandSoldering, symbol R_Small
- U1: footprint (none) -> SMD_fork:LGA-MPL3115A
Connections:
- net GND: now also J?.11, J?.4, J?.7, R?.2, R?.2
- net PD2: now also R?.1
- net PD3: now also J?.3, R?.1
- net RST: now also J?.9
- net RXD: now also J?.5
- net SCL: now also J?.2
- net SDA: now also J?.1
- net TXD: now also J?.6
- net VDD: now also J?.8
- net PD4: now reaches IC1.2 ((PCINT20/XCK/T0)PD4)
- net PD4: now also J?.10
- net PB6: no longer names the net of IC1.7 ((PCINT6/XTAL1/TOSC1)PB6)
- net PB7: no longer names the net of IC1.8 ((PCINT7/XTAL2/TOSC2)PB7)

Commit message: pcb added
Parts:
- removed J?: HEADER_1x11, symbol HEADER_1x11
- added J3: HEADER_1x09, Mlab_Pin_Headers:Angled_1x09, symbol HEADER_1x09
- added R6, R7, R8: 0, Capacitors_SMD:C_1206_HandSoldering, symbol R_Small
- gave numbers to parts that had none: 2
Connections:
- net PD4 is gone; now on net IGN: IC1.2 ((PCINT20/XCK/T0)PD4)
- net GND: now also J3.9, R6.1, R6.2, R8.1, R8.2
- net RST: now also J3.3
- net RXD: now also J3.4
- net SCL: now also J3.2
- net SDA: now also J3.1
- net TXD: now also J3.5
- net VDD: now also J3.8, R7.1, R7.2
- net PD2 renamed IGN
- net IGN: no longer IC1.32 ((PCINT18/INT0)PD2)
- net PD3 renamed IN
- net IN: now also IC1.32 ((PCINT18/INT0)PD2), J3.6; no longer IC1.1 ((PCINT19/OC2B/INT1)PD3)
- new net OUT: IC1.1 ((PCINT19/OC2B/INT1)PD3), J3.7
